File: ZM202_analog/analog_core.kicad_sch (KiCad schematic)
At the start: 41 parts, among them T1 BC846BLT1G, T2 BC856B, T3 BC846BLT1G, T4 BC846BLT1G, U10 TLC2272, U11 CD4052B, U7 LM358B, U8 TLC2272

Commit message: Finished first version of PCB. Added some capacitors at digital ICs.
Parts:
- added C17 (x4): C0603_100nF_25V, Capacitor_SMD:C_0603_1608Metric, symbol Jojos_Lib:C0603_100nF_25V
- T1, T3, T4: footprint SamacSys_Parts:SOT95P237X111-3N -> Package_TO_SOT_SMD:SOT-23
- T2: footprint SamacSys_Parts:SOT95P230X110-3N -> Package_TO_SOT_SMD:SOT-23
Connections:
- net +5V: now also C17.1, C17.1
- net -5V: now also C17.2, C17.2
- net GND: now also C17.1, C17.1, C17.2, C17.2
- net SN+: now also U8.3 (+); no longer U8.5 (+)
- net VIX: now also U8.7; no longer U8.1
- net VVX: now also U8.1; no longer U8.7
- net at R24.1, R27.1: now also U8.6 (-); no longer U8.2 (-)
- net at R25.1, R26.1: now also U8.5 (+); no longer U8.3 (+)
- net at U11.15: now also U8.2 (-); no longer U8.6 (-)
Other:
- moved on the sheet: U8A, U8B
